File: HW2/Custom Breakout/schematic_1.sch (EAGLE design)
At the start: 23 parts, among them J1 USB-MB-H

Commit message: Completed the part and connection schematic.
Parts:
- removed U$7: PICKIT3, custom:PICKIT3
Connections:
- removed net N$1: U$6.5.PGC, U$7.5.PGC
- removed net N$2: U$6.4.PGD, U$7.4.PGD
- removed net N$4: U$6.2.VDD, U$7.2.VDD
- removed net N$5: U$6.1.MCLR, U$7.1.MCLR
- new net A0: J2.8, U$1.2.A0
- new net A1: J2.7, U$1.3.A1
- new net A4/LED: J2.3, LED2.A, U$1.12.A4/LED
- new net B13: J3.6, U$1.24.B13
- new net B14: J3.7, U$1.25.B14
- new net B15: J3.8, U$1.26.B15
- new net B2: J2.6, U$1.6.B2
- new net B3: J2.5, U$1.7.B3
- new net B4/USER: J2.4, R1.1, U$1.11.B4/USER, U$5.1
- new net B7: J3.3, U$1.16.B7
- new net B8: J3.4, U$1.17.B8
- new net B9: J3.5, U$1.18.B9
- new net D+: J1.D+, U$1.21.D+/B10
- new net D-: J1.D-, U$1.22.D-/B11
- new net MCLR: R4.1, U$1.1.MCLR, U$4.1, U$6.1.MCLR
- new net N$7: C6.+, U$1.20.VCAP
- new net OSC1: U$1.9.OSC1/A2, U$8.1.OSC1
- new net OSC2: U$1.10.OSC2/A3, U$8.3.OSC2
- new net PGC: U$1.5.PGC/B1, U$6.5.PGC
- new net PGD: U$1.4.PGD/B0, U$6.4.PGD
- new net USBID: J1.ID, U$1.14.USBID/B5
- net +3V3: now also C3.1, C4.1, J2.2, R1.2, R4.2, U$1.13.VDD, U$1.23.VUSB3V3, U$1.28.AVDD, U$6.2.VDD
- net +5V: now also J3.2, U$1.15.VBUS
- net GND: now also C3.2, C4.2, C6.-, J2.1, J3.1, R3.1, U$1.19.VSS, U$1.27.AVSS, U$1.8.VSS, U$4.2, U$5.2, U$6.3.GND, U$8.2.GND
- net N$3: now also LED2.C, R3.2; no longer U$6.3.GND, U$7.3.GND
Other:
- moved on the sheet: C3, C4, C6, J2, J3, R1, R4, U$4, U$5, U$6, U$8
